Commit message: wip

File: referenceframe/urdf/testfiles/ur5_viam.urdf (robot description, URDF)
Before this commit: robot ur5, 8 links, 7 joints
Joints:
- joint wrist_1_joint: limit lower=-6.283185 upper=6.283185 effort=150 velocity=3.141592 -> lower=-6.283185 upper=6.283185 effort=28 velocity=3.141592
- joint wrist_2_joint: limit lower=-6.283185 upper=6.283185 effort=150 velocity=3.141592 -> lower=-6.283185 upper=6.283185 effort=28 velocity=3.141592
- joint wrist_3_joint: limit lower=-6.283185 upper=6.283185 effort=150 velocity=3.141592 -> lower=-6.283185 upper=6.283185 effort=28 velocity=3.141592

Commit message: modify the urdf for the ur5

File: referenceframe/urdf/testfiles/ur5_viam.urdf (robot description, URDF)
Before this commit: robot ur5, 8 links, 7 joints
Links:
- removed link world
- added link wrist_3_link; collision box size=0.08 0.17 0.08
- link base_link: geometry collision box size=0.151 0.151 0.240
- link forearm_link: geometry collision box size=0.100 0.100 0.490
- link upper_arm_link: geometry collision box size=0.130 0.130 0.550
- link wrist_1_link: geometry collision box size=0.080 0.20 0.080
- link wrist_2_link: geometry collision box size=0.08 0.08 0.20
Joints:
- removed joint base_joint
- added joint ee_fixed_joint: type revolute, parent wrist_3_link, child ee_link, origin xyz=0.0 0.0823 0.0 rpy=0.0 0.0 1.570796325, axis 0 1 0, limit lower=0 upper=0 effort=0.0 velocity=0
- joint elbow_joint: axis 0 -1 0 -> 0 1 0; limit lower=-3.141592 upper=3.141592 effort=150 velocity=3.141592 -> lower=-6.2831853 upper=6.2831853 effort=150.0 velocity=3.14159265; origin xyz=-0.3922 0.0 0.0 rpy=0.0 0.0 0.0 -> xyz=0.0 -0.1197 0.425 rpy=0.0 0.0 0.0
- joint shoulder_lift_joint: axis 0 -1 0 -> 0 1 0; limit lower=-6.283185 upper=6.283185 effort=150 velocity=3.141592 -> lower=-6.2831853 upper=6.2831853 effort=150.0 velocity=3.14159265; origin xyz=-0.425 0.0 0.0 rpy=0.0 0.0 0.0 -> xyz=0.0 0.13585 0.0 rpy=0.0 1.570796325 0.0
- joint shoulder_pan_joint: limit lower=-6.283185 upper=6.283185 effort=150 velocity=3.141592 -> lower=-6.2831853 upper=6.2831853 effort=150.0 velocity=3.14159265; origin xyz=0.0 0.0 0.1625 rpy=0.0 0.0 0.0 -> xyz=0.0 0.0 0.089159 rpy=0.0 0.0 0.0
- joint wrist_1_joint: axis 0 -1 0 -> 0 1 0; limit lower=-6.283185 upper=6.283185 effort=28 velocity=3.141592 -> lower=-3.14159265 upper=4.71 effort=28.0 velocity=3.14159265; origin xyz=0.0 -0.1333 0.0 rpy=0.0 0.0 0.0 -> xyz=0.0 0.0 0.39225 rpy=0.0 1.570796325 0.0
- joint wrist_2_joint: axis 0 0 -1 -> 0 0 1; limit lower=-6.283185 upper=6.283185 effort=28 velocity=3.141592 -> lower=-3.14159265 upper=4.71 effort=28.0 velocity=3.14159265; origin xyz=0.0 0.0 -0.0997 rpy=0.0 0.0 0.0 -> xyz=0.0 0.093 0.0 rpy=0.0 0.0 0.0
- joint wrist_3_joint: axis 0 -1 0 -> 0 1 0; child ee_link -> wrist_3_link; limit lower=-6.283185 upper=6.283185 effort=28 velocity=3.141592 -> lower=-3.14159265 upper=3.14159265 effort=28.0 velocity=3.14159265; origin xyz=0.0 -0.0996 0.0 rpy=1.5707963 0.0 0.0 -> xyz=0.0 0.0 0.09465 rpy=0.0 0.0 0.0

Commit message: actually good geometries

File: referenceframe/urdf/testfiles/ur5_viam.urdf (robot description, URDF)
Before this commit: robot ur5, 7 links, 6 joints
Links:
- removed link wrist_3_link
- added link ee_link
- added link world
- link base_link: geometry collision box size=0.120 0.120 0.260
- link forearm_link: geometry collision box size=0.090 0.130 0.130
- link shoulder_link: geometry collision box size=0.550 0.150 0.120
- link upper_arm_link: geometry collision box size=0.480 0.120 0.100
- link wrist_1_link: geometry 
- link wrist_2_link: geometry collision box size=0.080 0.150 0.100
Joints:
- added joint base_joint: type fixed, parent world, child base_link, origin xyz=0.0 0.0 0.0 rpy=0.0 0.0 0.0
- joint elbow_joint: axis 0 1 0 -> 0 -1 0; limit lower=-6.2831853 upper=6.2831853 effort=150.0 velocity=3.14159265 -> lower=-3.141592 upper=3.141592 effort=150 velocity=3.141592; origin xyz=0.0 -0.1197 0.425 rpy=0.0 0.0 0.0 -> xyz=-0.3922 0.0 0.0 rpy=0.0 0.0 0.0
- joint shoulder_lift_joint: axis 0 1 0 -> 0 -1 0; limit lower=-6.2831853 upper=6.2831853 effort=150.0 velocity=3.14159265 -> lower=-6.283185 upper=6.283185 effort=150 velocity=3.141592; origin xyz=0.0 0.13585 0.0 rpy=0.0 1.570796325 0.0 -> xyz=-0.425 0.0 0.0 rpy=0.0 0.0 0.0
- joint shoulder_pan_joint: limit lower=-6.2831853 upper=6.2831853 effort=150.0 velocity=3.14159265 -> lower=-6.283185 upper=6.283185 effort=150 velocity=3.141592; origin xyz=0.0 0.0 0.089159 rpy=0.0 0.0 0.0 -> xyz=0.0 0.0 0.1625 rpy=0.0 0.0 0.0
- joint wrist_1_joint: axis 0 1 0 -> 0 -1 0; limit lower=-3.14159265 upper=4.71 effort=28.0 velocity=3.14159265 -> lower=-6.283185 upper=6.283185 effort=28 velocity=3.141592; origin xyz=0.0 0.0 0.39225 rpy=0.0 1.570796325 0.0 -> xyz=0.0 -0.1333 0.0 rpy=0.0 0.0 0.0
- joint wrist_2_joint: axis 0 0 1 -> 0 0 -1; limit lower=-3.14159265 upper=4.71 effort=28.0 velocity=3.14159265 -> lower=-6.283185 upper=6.283185 effort=28 velocity=3.141592; origin xyz=0.0 0.093 0.0 rpy=0.0 0.0 0.0 -> xyz=0.0 0.0 -0.0997 rpy=0.0 0.0 0.0
- joint wrist_3_joint: axis 0 1 0 -> 0 -1 0; child wrist_3_link -> ee_link; limit lower=-3.14159265 upper=3.14159265 effort=28.0 velocity=3.14159265 -> lower=-6.283185 upper=6.283185 effort=28 velocity=3.141592; origin xyz=0.0 0.0 0.09465 rpy=0.0 0.0 0.0 -> xyz=0.0 -0.0996 0.0 rpy=1.5707963 0.0 0.0
