Commit message: rework the way we parse URDFs

File: referenceframe/urdf/testfiles/ur5e.urdf (robot description, URDF)
Before this commit: robot ur5, 8 links, 7 joints
Links:
- link forearm_link: geometry collision box size=0.480 0.120 0.100
- link shoulder_link: geometry 
- link upper_arm_link: geometry collision box size=0.550 0.150 0.120
- link wrist_1_link: geometry collision box size=0.090 0.130 0.130
- link wrist_2_link: geometry collision box size=0.080 0.180 0.100
Joints:
- joint elbow_joint: origin xyz=-0.3922 0.0 0.0 rpy=0.0 0.0 0.0 -> xyz=-0.425 0.0 0.0 rpy=0.0 0.0 0.0
- joint shoulder_lift_joint: origin xyz=-0.425 0.0 0.0 rpy=0.0 0.0 0.0 -> xyz=0.0 0.0 0.0 rpy=0.0 0.0 0.0
- joint wrist_1_joint: origin xyz=0.0 -0.1333 0.0 rpy=0.0 0.0 0.0 -> xyz=-.3922 -0.1333 0 rpy=0.0 0.0 0.0

Commit message: fix the final rotation

File: referenceframe/urdf/testfiles/ur5e.urdf (robot description, URDF)
Before this commit: robot ur5, 8 links, 7 joints
Links:
- added link wrist_3_link
Joints:
- added joint ee_joint: type fixed, parent wrist_3_link, child ee_link, origin xyz=0.0 0.0 0.0 rpy=1.5707963 0.0 0.0
- joint wrist_3_joint: child ee_link -> wrist_3_link; origin xyz=0.0 -0.0996 0.0 rpy=1.5707963 0.0 0.0 -> xyz=0.0 -0.0996 0.0 rpy=0.0 0.0 0.0

Commit message: RSDK-7435 fix the URDF conversion logic (#3562)

File: referenceframe/urdf/testfiles/ur5e.urdf (robot description, URDF)
Before this commit: robot ur5, 8 links, 7 joints
Links:
- added link wrist_3_link
- link wrist_2_link: geometry collision box size=0.080 0.180 0.100
Joints:
- added joint ee_joint: type fixed, parent wrist_3_link, child ee_link, origin xyz=0.0 0.0 0.0 rpy=1.5707963 0.0 0.0
- joint elbow_joint: origin xyz=-0.3922 0.0 0.0 rpy=0.0 0.0 0.0 -> xyz=-0.425 0.0 0.0 rpy=0.0 0.0 0.0
- joint shoulder_lift_joint: origin xyz=-0.425 0.0 0.0 rpy=0.0 0.0 0.0 -> xyz=0.0 0.0 0.0 rpy=0.0 0.0 0.0
- joint wrist_1_joint: origin xyz=0.0 -0.1333 0.0 rpy=0.0 0.0 0.0 -> xyz=-.3922 -0.1333 0 rpy=0.0 0.0 0.0
- joint wrist_3_joint: child ee_link -> wrist_3_link; origin xyz=0.0 -0.0996 0.0 rpy=1.5707963 0.0 0.0 -> xyz=0.0 -0.0996 0.0 rpy=0.0 0.0 0.0
